File: hw/mux.kicad_sch (KiCad schematic)
At the start: 3 parts, among them U14 BL1530TQFN

Commit message: ?
Parts:
- U14: JLCPCB_CORRECTION (none) -> 0;0;-90
Changed lines of the file:
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@@
+      (effects (font (size 1.27 1.27)) hide)
+    )
+    (property "JLCPCB_CORRECTION" "0;0;-90" (at 165.1 66.04 0)
       (effects (font (size 1.27 1.27)) hide)
     )
