File: hw/esp.kicad_sch (KiCad schematic)
At the start: 11 parts, among them SW2 EN, SW3 BOOT, U5 ESP32-S3-WROOM

Commit message: Mišmaš
Parts:
- C14, C15: Price (100ks) (none) -> 0.0029; Price (1ks) (none) -> 0.0029
- C16: Price (100ks) (none) -> 0.0159; Price (1ks) (none) -> 0.0159
- C17: Price (100ks) (none) -> 0.0011; Price (1ks) (none) -> 0.0011
- R20, R21, R23, R24: Price (100ks) (none) -> 0.0005; Price (1ks) (none) -> 0.0005
- SW2, SW3: LCSC C127488 -> C2985732; Price (100ks) (none) -> 0.0254; Price (1ks) (none) -> 0.0254
- U5: Price (100ks) (none) -> 4.9500; Price (1ks) (none) -> 6.2895
Changed lines of the file:
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@@
+      (effects (font (size 1.27 1.27)) hide)
+    )
+    (property "Price (100ks)" "0.0159" (at 180.34 40.64 0)
+      (effects (font (size 1.27 1.27)) hide)
+    )
+    (property "Price (1ks)" "0.0159" (at 180.34 40.64 0)
       (effects (font (size 1.27 1.27)) hide)
     )
@@
       (effects (font (size 1.27 1.27)) hide)
     )
+    (property "Price (100ks)" "0.0029" (at 132.08 93.98 0)
+      (effects (font (size 1.27 1.27)) hide)
+    )
+    (property "Price (1ks)" "0.0029" (at 132.08 93.98 0)
+      (effects (font (size 1.27 1.27)) hide)
+    )
     (pin "1")
     (pin "2")
@@
     )
     (property "Basic/Extended" "B" (at 142.24 55.88 0)
+      (effects (font (size 1.27 1.27)) hide)
+    )
+    (property "Price (100ks)" "0.0005" (at 142.24 55.88 0)
+      (effects (font (size 1.27 1.27)) hide)
+    )
+    (property "Price (1ks)" "0.0005" (at 142.24 55.88 0)
       (effects (font (size 1.27 1.27)) hide)
     )
@@
       (effects (font (size 1.27 1.27)) hide)
     )
-    (property "LCSC" "C127488" (at 139.7 129.54 0)
+    (property "LCSC" "C2985732" (at 139.7 129.54 0)
+      (effects (font (size 1.27 1.27)) hide)
+    )
+    (property "Price (100ks)" "0.0254" (at 139.7 129.54 0)
+      (effects (font (size 1.27 1.27)) hide)
+    )
+    (property "Price (1ks)" "0.0254" (at 139.7 129.54 0)
       (effects (font (size 1.27 1.27)) hide)
     )
@@
       (effects (font (size 1.27 1.27)) hide)
     )
+    (property "Price (100ks)" "0.0005" (at 114.3 93.98 0)
+      (effects (font (size 1.27 1.27)) hide)
+    )
+    (property "Price (1ks)" "0.0005" (at 114.3 93.98 0)
+      (effects (font (size 1.27 1.27)) hide)
+    )
     (pin "1")
     (pin "2")
@@
       (effects (font (size 1.27 1.27)) hide)
     )
+    (property "Price (100ks)" "0.0005" (at 132.08 69.85 0)
+      (effects (font (size 1.27 1.27)) hide)
+    )
+    (property "Price (1ks)" "0.0005" (at 132.08 69.85 0)
+      (effects (font (size 1.27 1.27)) hide)
+    )
     (pin "1")
     (pin "2")
@@
     )
     (property "Basic/Extended" "B" (at 121.92 93.98 0)
+      (effects (font (size 1.27 1.27)) hide)
+    )
+    (property "Price (100ks)" "0.0005" (at 121.92 93.98 0)
+      (effects (font (size 1.27 1.27)) hide)
+    )
+    (property "Price (1ks)" "0.0005" (at 121.92 93.98 0)
       (effects (font (size 1.27 1.27)) hide)
     )
@@
     )
     (property "JLCPCB_CORRECTION" "0;11.2;0" (at 179.07 55.88 0)
+      (effects (font (size 1.27 1.27)) hide)
+    )
+    (property "Price (100ks)" "4.9500" (at 179.07 55.88 0)
+      (effects (font (size 1.27 1.27)) hide)
+    )
+    (property "Price (1ks)" "6.2895" (at 179.07 55.88 0)
       (effects (font (size 1.27 1.27)) hide)
     )
@@
       (effects (font (size 1.27 1.27)) hide)
     )
-    (property "LCSC" "C127488" (at 127 129.54 0)
+    (property "LCSC" "C2985732" (at 127 129.54 0)
+      (effects (font (size 1.27 1.27)) hide)
+    )
+    (property "Price (100ks)" "0.0254" (at 127 129.54 0)
+      (effects (font (size 1.27 1.27)) hide)
+    )
+    (property "Price (1ks)" "0.0254" (at 127 129.54 0)
       (effects (font (size 1.27 1.27)) hide)
     )
@@
     )
     (property "info" "25V, X5R" (at 142.24 93.98 0)
+      (effects (font (size 1.27 1.27)) hide)
+    )
+    (property "Price (100ks)" "0.0029" (at 142.24 93.98 0)
+      (effects (font (size 1.27 1.27)) hide)
+    )
+    (property "Price (1ks)" "0.0029" (at 142.24 93.98 0)
       (effects (font (size 1.27 1.27)) hide)
     )
@@
       (effects (font (size 1.27 1.27)) hide)
     )
+    (property "Price (100ks)" "0.0011" (at 180.34 45.72 0)
+      (effects (font (size 1.27 1.27)) hide)
+    )
+    (property "Price (1ks)" "0.0011" (at 180.34 45.72 0)
+      (effects (font (size 1.27 1.27)) hide)
+    )

Commit message: Resolves #69 Change from ESP32-S3 with octcal SPIRAM to quad SPIRAM
Parts:
- U5: LCSC C2913202 -> C2913205; info ESP32-S3-WROOM-1-N16R8 -> ESP32-S3-WROOM-1-N16R2
Other:
- moved on the sheet: C14, R20, R21, R23

Commit message: PCB
Parts:
- U5: LCSC C2913205 -> C2913204; info ESP32-S3-WROOM-1-N16R2 -> ESP32-S3-WROOM-1-N8R2
Changed lines of the file:
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@@
       (effects (font (size 1.27 1.27)) hide)
     )
-    (property "LCSC" "C2913205" (at 179.07 43.18 0)
+    (property "LCSC" "C2913204" (at 179.07 43.18 0)
       (effects (font (size 1.27 1.27)) hide)
     )
@@
       (effects (font (size 1.27 1.27)) hide)
     )
-    (property "info" "ESP32-S3-WROOM-1-N16R2" (at 179.07 36.83 0)
+    (property "info" "ESP32-S3-WROOM-1-N8R2" (at 179.07 36.83 0)
       (effects (font (size 1.27 1.27)) hide)
     )

Commit message: D7 and bigger vias
Parts:
- SW2, SW3: LCSC C2985732 -> C115360
Changed lines of the file:
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@@
       (effects (font (size 1.27 1.27)) hide)
     )
-    (property "LCSC" "C2985732" (at 139.7 129.54 0)
+    (property "LCSC" "C115360" (at 139.7 129.54 0)
       (effects (font (size 1.27 1.27)) hide)
     )
@@
       (effects (font (size 1.27 1.27)) hide)
     )
-    (property "LCSC" "C2985732" (at 127 129.54 0)
-      (effects (font (size 1.27 1.27)) hide)
-    )
+    (property "LCSC" "C115360" (at 127 129.54 0)
+      (effects (font (size 1.27 1.27)) hide)
+    )
